File: pcb/WindTurbineController.kicad_pcb (KiCad board)
At the start: 2 copper layers, 60 x 25 mm, 33 parts, among them IC1 DRV8220DSGR, IC2 DRV8220DSGR, J1 Conn_01x02, J2 Conn_01x02, J3 Conn_01x04, J4 Conn_01x02, J5 Conn_01x04, J6 Conn_01x01, J7 Conn_01x01, U1 MUBv1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

Commit message: fixes
Parts:
- removed C10, C11, C7: 100nF, Capacitor_SMD:C_0603_1608Metric
- removed C8, C9: 10uF, Capacitor_SMD:C_0805_2012Metric
- removed D3: SBT55LAFC, custom_parts:SMAF-C
- moved L1 6.19 mm to (85.5, 76.0), turned to -90 degrees
Connections:
- net Net-(L1-Pad2) renamed /IND_IN
- J1 pad 1: Net-(IC1-Pad3) -> Net-(IC1-OUT2)
- J1 pad 2: Net-(IC1-Pad2) -> Net-(IC1-OUT1)
- J2 pad 1: Net-(IC2-Pad3) -> Net-(IC2-OUT2)
- J2 pad 2: Net-(IC2-Pad2) -> Net-(IC2-OUT1)
Routing:
- net /IND_IN: track 31.8 -> 10.7 mm, vias 1 -> 4
- net Net-(IC1-Pad2): track 5.93 -> 0.00 mm
- net Net-(IC1-OUT1): track 0.00 -> 5.93 mm
- net Net-(IC1-Pad3): track 4.03 -> 0.00 mm
- net Net-(IC1-OUT2): track 0.00 -> 4.03 mm
- net +12V: track 70.4 -> 66.5 mm, vias 3 -> 7
- net Net-(IC2-Pad2): track 3.14 -> 0.00 mm
- net Net-(IC2-OUT1): track 0.00 -> 3.14 mm
- added copper zone on B.Cu, net +12V
- added copper zone on B.Cu, net /IND_IN
- added copper zone on F.Cu, net /IND_IN
- added copper zone on F.Cu, net GND
