File: pcb/WindTurbineController.kicad_sch (KiCad schematic)
At the start: 33 parts, among them IC1 DRV8220DSGR, IC2 DRV8220DSGR, J1 Conn_01x02, J2 Conn_01x02, J3 Conn_01x04, J4 Conn_01x02, J5 Conn_01x04, J6 Conn_01x01, J7 Conn_01x01, U1 MUBv1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

Commit message: fixes
Parts:
- ?: renamed from C3; value 10uF -> (none); footprint Capacitor_SMD:C_0805_2012Metric -> (none)
- ?: renamed from U1; value MUBv1 -> (none); footprint MUB:MUB_v1 -> (none)
- ?: renamed from IC1; value DRV8220DSGR -> (none); footprint SON50P200X200X80-9N -> (none)
- ?: renamed from R3; value 100k -> (none); footprint Resistor_SMD:R_0603_1608Metric -> (none)
- ?: renamed from R1; value 11.3k -> (none); footprint Resistor_SMD:R_0603_1608Metric -> (none)
- ?: renamed from J5; value Conn_01x04 -> (none); footprint Connector_PinHeader_2.54mm:PinHeader_1x04_P2.54mm_Vertical -> (none)
- ?: renamed from C2; value 10uF -> (none); footprint Capacitor_SMD:C_0805_2012Metric -> (none)
- ?: renamed from C9; value 10uF -> (none); footprint Capacitor_SMD:C_0805_2012Metric -> (none)
- ?: renamed from J4; value Conn_01x02 -> (none); footprint Connector_PinHeader_2.54mm:PinHeader_1x02_P2.54mm_Vertical -> (none)
- ?: renamed from J3; value Conn_01x04 -> (none); footprint Connector_PinHeader_2.54mm:PinHeader_1x04_P2.54mm_Vertical -> (none)
- ?: renamed from R4; value 11.3k -> (none); footprint Resistor_SMD:R_0603_1608Metric -> (none)
- ?: renamed from C1; value 220uF -> (none); footprint Capacitor_THT:C_Radial_D10.0mm_H16.0mm_P5.00mm -> (none)
- ?: renamed from C5; value 10nF -> (none); footprint Capacitor_SMD:C_0402_1005Metric -> (none)
- ?: renamed from C4; value 82pF -> (none); footprint Capacitor_SMD:C_0402_1005Metric -> (none)
- ?: renamed from U3; value TLV493D -> (none); footprint Package_TO_SOT_SMD:SOT-23-6 -> (none)
- ?: renamed from D1; value D_Bridge_+-AA -> (none); footprint Package_TO_SOT_SMD:TO-269AA -> (none)
- ?: renamed from IC2; value DRV8220DSGR -> (none); footprint SON50P200X200X80-9N -> (none)
- ?: renamed from D2; value D_Bridge_+-AA -> (none); footprint Package_TO_SOT_SMD:TO-269AA -> (none)
- ?: renamed from U4; value AH1388 -> (none); footprint custom_parts:X2-DFN1410-4 -> (none)
- ?: renamed from C6; value 10uF -> (none); footprint Capacitor_SMD:C_0805_2012Metric -> (none)
- ?: renamed from U2; value TLV493D -> (none); footprint Package_TO_SOT_SMD:SOT-23-6 -> (none)
- ?: renamed from D3; value SBT55LAFC -> (none); footprint custom_parts:SMAF-C -> (none)
- ?: renamed from J2; value Conn_01x02 -> (none); footprint Connector_PinHeader_2.54mm:PinHeader_1x02_P2.54mm_Vertical -> (none)
- ?: renamed from C7; value 100nF -> (none); footprint Capacitor_SMD:C_0603_1608Metric -> (none)
- ?: renamed from R2; value 11.3k -> (none); footprint Resistor_SMD:R_0603_1608Metric -> (none)
- ?: renamed from C11; value 100nF -> (none); footprint Capacitor_SMD:C_0603_1608Metric -> (none)
- ?: renamed from L1; value 32.5uH -> (none); footprint custom_parts:PCC-M105xx -> (none)
- ?: renamed from C10; value 100nF -> (none); footprint Capacitor_SMD:C_0603_1608Metric -> (none)
- ?: renamed from U5; value RT8279GSP -> (none); footprint Package_SO:SOIC-8-1EP_3.9x4.9mm_P1.27mm_EP2.514x3.2mm -> (none)
- ?: renamed from J1; value Conn_01x02 -> (none); footprint Connector_PinHeader_2.54mm:PinHeader_1x02_P2.54mm_Vertical -> (none)
- ?: renamed from J7; value Conn_01x01 -> (none); footprint MountingHole:MountingHole_2.2mm_M2 -> (none)
- ?: renamed from J6; value Conn_01x01 -> (none); footprint MountingHole:MountingHole_2.2mm_M2 -> (none)
- ?: renamed from C8; value 10uF -> (none); footprint Capacitor_SMD:C_0805_2012Metric -> (none)
Connections:
- net IND_IN: now reaches ?.1, ?.1 (BOOT), ?.1 (K), ?.2
